Commit message: Rename thumb_mcp

File: ros2/telekinesis/telekinesis/leap_hand_mesh_right/robot_pybullet.urdf (robot description, URDF)
Before this commit: robot onshape, 21 links, 20 joints
Links:
- removed link pip_4
- added link thumb_mcp, mass 0.032; collision mesh filename=pip.stl; visual mesh filename=pip.stl
Joints:
- joint 12: child pip_4 -> thumb_mcp
- joint 13: parent pip_4 -> thumb_mcp

Commit message: Reordered joint indices. Need to figure out the offset of the palm (where the origin is of the URDF)

File: ros2/telekinesis/telekinesis/leap_hand_mesh_right/robot_pybullet.urdf (robot description, URDF)
Before this commit: robot onshape, 21 links, 20 joints
Links:
- removed link realtip
- removed link realtip_2
- removed link realtip_3
- removed link realtip_4
Joints:
- removed joint 16
- removed joint 17
- removed joint 18
- removed joint 19
